File: LM2596HV_breakout.kicad_pcb (KiCad board)
At the start: 2 copper layers, 50 x 30 mm, 11 parts, among them J1 Screw_Terminal_01x02, J2 Screw_Terminal_01x02, U1 LM2596HVS

Commit message: update,
Parts:
- J1: value Screw_Terminal_01x02 -> VIN
- J2: value Screw_Terminal_01x02 -> VOUT
- moved R2 0.53 mm to (36.9, 35.8)
- turned J1 to 180 degrees
- turned J2 to 180 degrees
- turned L1 to 0 degrees
Connections:
- J1 pad 1: VIN -> GND
- J1 pad 2: GND -> VIN
- J2 pad 1: VOUT -> GND
- J2 pad 2: GND -> VOUT
Routing:
- net Net-(L1-Pad1): track 51.9 -> 44.1 mm
- net GND: track 129.9 -> 134.9 mm
- net Net-(R1-Pad2): track 14.7 -> 19.6 mm
- net VOUT: track 44.3 -> 48.6 mm
- net VIN: track 37.6 -> 38.5 mm

Commit message: update,
Parts:
- added D2: LED_GREEN, LED_SMD:LED_0805_2012Metric_Pad1.15x1.40mm_HandSolder, F.Cu at (39.7, 17.7)
- added R3: R511, Resistor_SMD:R_0805_2012Metric_Pad1.15x1.40mm_HandSolder, F.Cu at (43.2, 17.8)
- J1, J2: footprint w_conn_mpt:mpt_0,5%2f2-2,54 -> footprint-lib:mpt_0,5%2f2-2,54
- moved J2 23.0 mm to (53.6, 40.3), turned to 270 degrees
- moved J1 21.0 mm to (19.8, 40.0), turned to 270 degrees
- moved R1 18.4 mm to (46.6, 17.8), turned to 90 degrees
- moved R2 18.1 mm to (36.2, 17.8), turned to 90 degrees
- moved C3 15.7 mm to (37.4, 40.0), turned to 180 degrees
- moved C4 13.4 mm to (45.8, 38.7)
- moved D1 11.1 mm to (37.8, 35.3), turned to 0 degrees
- moved U1 11.1 mm to (25.2, 21.6), turned to 180 degrees
- moved L1 8.99 mm to (41.5, 26.7), turned to 90 degrees
- moved C2 8.81 mm to (31.0, 28.9), turned to 0 degrees
- moved C1 7.72 mm to (29.0, 36.8)
Connections:
- L1 pad 1: Net-(L1-Pad1) -> Net-(D1-Pad1)
- U1 pad 2: Net-(L1-Pad1) -> Net-(D1-Pad1)
Routing:
- net Net-(L1-Pad1): track 44.1 -> 0.00 mm
- net Net-(D1-Pad1): track 0.00 -> 17.4 mm
- net VIN: track 38.5 -> 22.7 mm
- net VOUT: track 48.6 -> 40.3 mm
- net Net-(D2-Pad2): track 0.00 -> 3.49 mm
- net GND: track 134.9 -> 137.4 mm
- net Net-(R1-Pad2): track 19.6 -> 20.2 mm

Commit message: update,
Parts:
- moved J2 24.7 mm to (42.2, 18.4), turned to 90 degrees
- moved C3 22.0 mm to (36.5, 18.1), turned to 90 degrees
- moved R1 17.8 mm to (29.2, 21.5)
- moved C2 15.6 mm to (17.6, 37.0)
- moved R3 11.5 mm to (32.4, 21.7)
- moved D1 7.53 mm to (32.5, 30.0), turned to 270 degrees
- moved D2 7.15 mm to (32.6, 17.3), turned to 270 degrees
- moved R2 7.11 mm to (29.1, 17.2), turned to 270 degrees
- moved U1 4.56 mm to (21.3, 23.9), turned to 90 degrees
- moved C4 4.54 mm to (41.3, 39.4), turned to 0 degrees
- moved C1 2.43 mm to (28.1, 39.1), turned to 0 degrees
- moved J1 2.39 mm to (18.4, 41.9), turned to 0 degrees
- moved L1 1.88 mm to (41.7, 28.6)
Routing:
- net Net-(D1-Pad1): track 17.4 -> 31.4 mm
- net Net-(R1-Pad2): track 20.2 -> 25.9 mm
- net VIN: track 22.7 -> 27.3 mm
- net VOUT: track 40.3 -> 38.0 mm
- net Net-(D2-Pad2): track 3.49 -> 1.69 mm
- net GND: track 137.4 -> 136.8 mm

Commit message: update,
Parts:
- moved C4 12.0 mm to (41.9, 27.4)
- moved L1 9.54 mm to (42.1, 38.1)
- moved C2 3.06 mm to (17.2, 34.0), turned to 180 degrees
- moved C3 1.53 mm to (35.3, 17.2)
- moved J1 1.09 mm to (18.4, 40.8), turned to 180 degrees
- moved D2 0.37 mm to (32.2, 17.2)
- moved R3 0.29 mm to (32.2, 21.5)
- moved J2 0.22 mm to (42.3, 18.1)
- moved R1 0.10 mm to (29.1, 21.5)
Routing:
- net VIN: track 27.3 -> 18.5 mm
- net Net-(D1-Pad1): track 31.4 -> 36.3 mm
- net Net-(D2-Pad2): track 1.69 -> 4.07 mm
- net GND: track 136.8 -> 138.1 mm

Commit message: update,
Parts:
- moved D2 2.81 mm to (32.2, 20.0)
- moved C3 2.81 mm to (35.2, 20.0)
- moved R1 2.81 mm to (29.1, 24.3)
- moved R2 2.81 mm to (29.1, 20.0)
- moved R3 2.81 mm to (32.1, 24.3)
- moved C2 2.29 mm to (18.1, 36.1)
- turned D1 to 90 degrees
- turned J1 to 0 degrees
Connections:
- J1 pad 1: GND -> VIN
- J1 pad 2: VIN -> GND
Routing:
- net VIN: track 18.5 -> 26.1 mm
- net GND: track 138.1 -> 145.0 mm
- net Net-(D1-Pad1): track 36.3 -> 30.3 mm
- net Net-(D2-Pad2): track 4.07 -> 2.22 mm
- net Net-(R1-Pad2): track 25.9 -> 25.2 mm
